Commit message: fix IK

File: fetch_description/robots/fetch_obj.urdf (robot description, URDF)
Before this commit: robot fetch, 26 links, 25 joints
Joints:
- joint head_pan_joint: type revolute -> fixed
- joint head_tilt_joint: type revolute -> fixed
- joint l_wheel_joint: type continuous -> fixed
- joint r_wheel_joint: type continuous -> fixed
- joint shoulder_lift_joint: limit lower=-1.221 upper=1.518 effort=131.76 velocity=1.454 -> lower=-0.2 upper=0.1 effort=131.76 velocity=1.454
- joint torso_lift_joint: type prismatic -> fixed
- joint upperarm_roll_joint: limit effort=76.94 velocity=1.571 -> lower=1.3 upper=1.7 effort=76.94 velocity=1.571; type continuous -> revolute
