Commit message: pick up blocks

File: fetch_description/robots/fetch.urdf (robot description, URDF)
Before this commit: robot fetch, 26 links, 25 joints
Joints:
- joint head_pan_joint: type revolute -> fixed
- joint head_tilt_joint: type revolute -> fixed
- joint l_wheel_joint: type continuous -> fixed
- joint r_wheel_joint: type continuous -> fixed
- joint torso_lift_joint: type prismatic -> fixed

File: fetch_description/robots/fetch_obj.urdf (robot description, URDF)
Before this commit: robot fetch, 26 links, 25 joints
Joints:
- joint shoulder_lift_joint: limit lower=-0.2 upper=0.1 effort=131.76 velocity=1.454 -> lower=-0.5 upper=1.518 effort=131.76 velocity=1.454
